Commit message: WIP transition planning
Some start conf in collision. First conf in the ladder graph jumps.

File: src/compas_fab/data/universal_robot/ur_description/urdf/ur5.urdf (robot description, URDF)
Before this commit: robot ur5, 11 links, 10 joints
Joints:
- joint elbow_joint: limit lower=-6.2831853 upper=6.2831853 effort=150.0 velocity=3.15 -> lower=-3.1415926 upper=3.1415926 effort=150.0 velocity=3.15
