Commit message: rebuild UR3 urdf with dae descriptions.
The transition planning self-collision between element and the robot body bug persists.

File: src/compas_fab/data/universal_robot/ur_description/urdf/ur3.urdf (robot description, URDF)
Before this commit: robot ur3, 11 links, 10 joints
Links:
- link base_link: geometry collision mesh filename=package://ur_description/meshes/ur3/collision/base.stl; visual mesh filename=package://ur_description/meshes/ur3/visual/base.dae
- link forearm_link: geometry collision mesh filename=package://ur_description/meshes/ur3/collision/forearm.stl; visual mesh filename=package://ur_description/meshes/ur3/visual/forearm.dae
- link shoulder_link: geometry collision mesh filename=package://ur_description/meshes/ur3/collision/shoulder.stl; visual mesh filename=package://ur_description/meshes/ur3/visual/shoulder.dae
- link upper_arm_link: geometry collision mesh filename=package://ur_description/meshes/ur3/collision/upperarm.stl; visual mesh filename=package://ur_description/meshes/ur3/visual/upperarm.dae
- link wrist_1_link: geometry collision mesh filename=package://ur_description/meshes/ur3/collision/wrist1.stl; visual mesh filename=package://ur_description/meshes/ur3/visual/wrist1.dae
- link wrist_2_link: geometry collision mesh filename=package://ur_description/meshes/ur3/collision/wrist2.stl; visual mesh filename=package://ur_description/meshes/ur3/visual/wrist2.dae
- link wrist_3_link: geometry collision mesh filename=package://ur_description/meshes/ur3/collision/wrist3.stl; visual mesh filename=package://ur_description/meshes/ur3/visual/wrist3.dae
